File: badgePCB/badgePCB.kicad_sch (KiCad schematic)
At the start: 26 parts, among them SW1 TS-1187A-B-A-B, SW2 TS-1187A-B-A-B, SW3 TS-1187A-B-A-B, U1 XIAO-ESP32-C3-DIP

Commit message: fix schm
Parts:
- added R10, R9: 100R, Resistor_SMD:R_0603_1608Metric_Pad0.98x0.95mm_HandSolder, symbol Device:R
- R1, R2, R3, R4, R5, R6, R7, R8: value R -> 100R; LCSC Part (none) -> C22775
- U1: footprint Module:MOUDLE14P-XIAO-DIP-SMD -> XIAO:XIAO-ESP32C3-DIP
Connections:
- net GND: now also R10.2, R9.2; no longer R7.1, R8.1
- net MID1: now also R2.2; no longer R3.2
- net MID3: now also R3.2; no longer R2.2
- net at D1.1 (K), D2.2 (A), D3.2 (A)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: now also R2.1; no longer R3.1
- net at D3.1 (K), D4.2 (A), D5.1 (K)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: now also R3.1; no longer R2.1
- net at D14.1 (K): now also R8.1; no longer R8.2
- net at R7.2: now also R10.1; no longer D13.1 (K)
- new net: R8.2, R9.1
- new net: D13.1 (K), R7.1
- no-connect marks 0 -> 2

Commit message: koi
Parts:
- U1: footprint XIAO:XIAO-ESP32C3-DIP -> XIAO:XIAO-ESP32C3-SMD
Changed lines of the file:
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@@
 			)
 		)
-		(property "Footprint" "XIAO:XIAO-ESP32C3-DIP"
+		(property "Footprint" "XIAO:XIAO-ESP32C3-SMD"
 			(at 95.504 133.604 0)
 			(hide yes)

Commit message: finishPCB
Parts:
- D1, D10, D11, D12, D13, D14, D2, D3, D4, D5, D6, D7, D8, D9: footprint LED_SMD:LED_0805_2012Metric_Pad1.15x1.40mm_HandSolder -> Extra:LED_0805_2012Metric_Pad1.15x1.40mm_HandSolder
Connections:
- net MID1: now also U1.2 (GPIO3/A1/D1); no longer U1.1 (GPIO2/A0/D0)
- net MID2: now also U1.3 (GPIO4/A2/D2); no longer U1.2 (GPIO3/A1/D1)
- net MID3: now also U1.1 (GPIO2/A0/D0); no longer U1.3 (GPIO4/A2/D2)
Changed lines of the file:
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@@
 		)
 	)
-	(global_label "MID3"
+	(global_label "MID2"
 		(shape input)
-		(at 76.2 114.3 180)
+		(at 45.72 53.34 270)
 		(fields_autoplaced yes)
 		(effects
@@
 		)
 		(property "Intersheetrefs" "${INTERSHEET_REFS}"
-			(at 68.6791 114.3 0)
+			(at 45.72 60.8609 90)
 			(hide yes)
 			(show_name no)
@@
 	(global_label "MID2"
 		(shape input)
-		(at 45.72 53.34 270)
+		(at 76.2 114.3 180)
 		(fields_autoplaced yes)
 		(effects
@@
 		)
 		(property "Intersheetrefs" "${INTERSHEET_REFS}"
-			(at 45.72 60.8609 90)
+			(at 68.6791 114.3 0)
 			(hide yes)
 			(show_name no)
@@
 		)
 	)
-	(global_label "IDUp"
+	(global_label "MID1"
 		(shape input)
-		(at 114.3 125.73 0)
+		(at 76.2 110.49 180)
 		(fields_autoplaced yes)
 		(effects
@@
 				(size 1.27 1.27)
 			)
-			(justify left)
+			(justify right)
 		)
 		(property "Intersheetrefs" "${INTERSHEET_REFS}"
-			(at 121.6395 125.73 0)
+			(at 68.6791 110.49 0)
 			(hide yes)
 			(show_name no)
@@
 					(size 1.27 1.27)
 				)
-				(justify left)
+				(justify right)
 			)
 		)
 	)
-	(global_label "SID1"
+	(global_label "IDUp"
 		(shape input)
-		(at 76.2 118.11 180)
+		(at 114.3 125.73 0)
 		(fields_autoplaced yes)
 		(effects
@@
 				(size 1.27 1.27)
 			)
-			(justify right)
+			(justify left)
 		)
 		(property "Intersheetrefs" "${INTERSHEET_REFS}"
-			(at 68.921 118.11 0)
+			(at 121.6395 125.73 0)
 			(hide yes)
 			(show_name no)
@@
 					(size 1.27 1.27)
 				)
-				(justify right)
+				(justify left)
 			)
 		)
 	)
-	(global_label "SLED"
+	(global_label "SID1"
 		(shape input)
-		(at 114.3 129.54 0)
+		(at 76.2 118.11 180)
 		(fields_autoplaced yes)
 		(effects
@@
 				(size 1.27 1.27)
 			)
-			(justify left)
+			(justify right)
 		)
 		(property "Intersheetrefs" "${INTERSHEET_REFS}"
-			(at 121.9418 129.54 0)
+			(at 68.921 118.11 0)
 			(hide yes)
 			(show_name no)
@@
 					(size 1.27 1.27)
 				)
-				(justify left)
+				(justify right)
 			)
 		)
 	)
-	(global_label "MID1"
+	(global_label "SLED"
 		(shape input)
-		(at 76.2 106.68 180)
+		(at 114.3 129.54 0)
 		(fields_autoplaced yes)
 		(effects
@@
 				(size 1.27 1.27)
 			)
-			(justify right)
+			(justify left)
 		)
 		(property "Intersheetrefs" "${INTERSHEET_REFS}"
-			(at 68.6791 106.68 0)
+			(at 121.9418 129.54 0)
 			(hide yes)
 			(show_name no)
@@
 					(size 1.27 1.27)
 				)
-				(justify right)
+				(justify left)
 			)
 		)
@@
 		)
 	)
-	(global_label "Action"
+	(global_label "MID3"
 		(shape input)
-		(at 99.06 165.1 0)
+		(at 76.2 106.68 180)
 		(fields_autoplaced yes)
 		(effects
@@
 				(size 1.27 1.27)
 			)
-			(justify left)
+			(justify right)
 		)
 		(property "Intersheetrefs" "${INTERSHEET_REFS}"
-			(at 107.8509 165.1 0)
+			(at 68.6791 106.68 0)
 			(hide yes)
 			(show_name no)
@@
 					(size 1.27 1.27)
 				)
-				(justify left)
+				(justify right)
 			)
 		)
 	)
-	(global_label "IDDown"
+	(global_label "Action"
 		(shape input)
-		(at 114.3 121.92 0)
+		(at 99.06 165.1 0)
 		(fields_autoplaced yes)
 		(effects
@@
 		)
 		(property "Intersheetrefs" "${INTERSHEET_REFS}"
-			(at 124.0585 121.92 0)
+			(at 107.8509 165.1 0)
 			(hide yes)
 			(show_name no)
@@
 		)
 	)
-	(global_label "SID2"
+	(global_label "IDDown"
 		(shape input)
-		(at 76.2 121.92 180)
+		(at 114.3 121.92 0)
 		(fields_autoplaced yes)
 		(effects
@@
 				(size 1.27 1.27)
 			)
-			(justify right)
+			(justify left)
 		)
 		(property "Intersheetrefs" "${INTERSHEET_REFS}"
-			(at 68.921 121.92 0)
+			(at 124.0585 121.92 0)
 			(hide yes)
 			(show_name no)
@@
 					(size 1.27 1.27)
 				)
-				(justify right)
+				(justify left)
 			)
 		)
 	)
-	(global_label "MID2"
+	(global_label "SID2"
 		(shape input)
-		(at 76.2 110.49 180)
+		(at 76.2 121.92 180)
 		(fields_autoplaced yes)
 		(effects
@@
 		)
 		(property "Intersheetrefs" "${INTERSHEET_REFS}"
-			(at 68.6791 110.49 0)
+			(at 68.921 121.92 0)
 			(hide yes)
 			(show_name no)
@@
 			)
 		)
-		(property "Footprint" "LED_SMD:LED_0805_2012Metric_Pad1.15x1.40mm_HandSolder"
+		(property "Footprint" "Extra:LED_0805_2012Metric_Pad1.15x1.40mm_HandSolder"
 			(at 38.1 40.64 0)
 			(hide yes)
@@
 			)
 		)
-		(property "Footprint" "LED_SMD:LED_0805_2012Metric_Pad1.15x1.40mm_HandSolder"
+		(property "Footprint" "Extra:LED_0805_2012Metric_Pad1.15x1.40mm_HandSolder"
 			(at 45.72 30.48 0)
 			(hide yes)
@@
 			)
 		)
-		(property "Footprint" "LED_SMD:LED_0805_2012Metric_Pad1.15x1.40mm_HandSolder"
+		(property "Footprint" "Extra:LED_0805_2012Metric_Pad1.15x1.40mm_HandSolder"
 			(at 124.46 34.29 0)
 			(hide yes)
@@
 			)
 		)
-		(property "Footprint" "LED_SMD:LED_0805_2012Metric_Pad1.15x1.40mm_HandSolder"
+		(property "Footprint" "Extra:LED_0805_2012Metric_Pad1.15x1.40mm_HandSolder"
 			(at 53.34 40.64 0)
 			(hide yes)
@@
 			)
 		)
-		(property "Footprint" "LED_SMD:LED_0805_2012Metric_Pad1.15x1.40mm_HandSolder"
+		(property "Footprint" "Extra:LED_0805_2012Metric_Pad1.15x1.40mm_HandSolder"
 			(at 25.4 82.55 0)
 			(hide yes)
@@
 			)
 		)
-		(property "Footprint" "LED_SMD:LED_0805_2012Metric_Pad1.15x1.40mm_HandSolder"
+		(property "Footprint" "Extra:LED_0805_2012Metric_Pad1.15x1.40mm_HandSolder"
 			(at 38.1 45.72 0)
 			(hide yes)
@@
 			)
 		)
-		(property "Footprint" "LED_SMD:LED_0805_2012Metric_Pad1.15x1.40mm_HandSolder"
+		(property "Footprint" "Extra:LED_0805_2012Metric_Pad1.15x1.40mm_HandSolder"
 			(at 45.72 35.56 0)
 			(hide yes)
@@
 			)
 		)
-		(property "Footprint" "LED_SMD:LED_0805_2012Metric_Pad1.15x1.40mm_HandSolder"
+		(property "Footprint" "Extra:LED_0805_2012Metric_Pad1.15x1.40mm_HandSolder"
 			(at 116.84 39.37 0)
 			(hide yes)
@@
 			)
 		)
-		(property "Footprint" "LED_SMD:LED_0805_2012Metric_Pad1.15x1.40mm_HandSolder"
+		(property "Footprint" "Extra:LED_0805_2012Metric_Pad1.15x1.40mm_HandSolder"
 			(at 44.45 82.55 0)
 			(hide yes)
@@
 			)
 		)
-		(property "Footprint" "LED_SMD:LED_0805_2012Metric_Pad1.15x1.40mm_HandSolder"
+		(property "Footprint" "Extra:LED_0805_2012Metric_Pad1.15x1.40mm_HandSolder"
 			(at 53.34 45.72 0)
 			(hide yes)
@@
 			)
 		)
-		(property "Footprint" "LED_SMD:LED_0805_2012Metric_Pad1.15x1.40mm_HandSolder"
+		(property "Footprint" "Extra:LED_0805_2012Metric_Pad1.15x1.40mm_HandSolder"
 			(at 116.84 44.45 0)
 			(hide yes)
@@
 			)
 		)
-		(property "Footprint" "LED_SMD:LED_0805_2012Metric_Pad1.15x1.40mm_HandSolder"
+		(property "Footprint" "Extra:LED_0805_2012Metric_Pad1.15x1.40mm_HandSolder"
 			(at 132.08 44.45 0)
 			(hide yes)
@@
 			)
 		)
-		(property "Footprint" "LED_SMD:LED_0805_2012Metric_Pad1.15x1.40mm_HandSolder"
+		(property "Footprint" "Extra:LED_0805_2012Metric_Pad1.15x1.40mm_HandSolder"
 			(at 124.46 29.21 0)
 			(hide yes)
@@
 			)
 		)
-		(property "Footprint" "LED_SMD:LED_0805_2012Metric_Pad1.15x1.40mm_HandSolder"
+		(property "Footprint" "Extra:LED_0805_2012Metric_Pad1.15x1.40mm_HandSolder"
 			(at 132.08 39.37 0)
 			(hide yes)
