File: badgePCB/badgePCB.kicad_pcb (KiCad board)
At the start: 2 copper layers, 54 x 38.5 mm, 28 parts, among them SW1 TS-1187A-B-A-B, SW2 TS-1187A-B-A-B, SW3 TS-1187A-B-A-B, U1 XIAO-ESP32-C3-DIP

Commit message: routing
Routing:
- net SID3: track 0.00 -> 36.3 mm, vias 0 -> 1
- net SID2: track 0.00 -> 35.0 mm, vias 0 -> 1
- net Net-(D1-K): track 0.00 -> 34.5 mm, vias 0 -> 2
- net SID1: track 0.00 -> 33.6 mm, vias 0 -> 1
- net MID3: track 0.00 -> 33.4 mm, vias 0 -> 1
- net MID1: track 0.00 -> 32.5 mm, vias 0 -> 1
- net Net-(D11-K): track 0.00 -> 31.6 mm
- net Action: track 0.00 -> 30.8 mm
- net Net-(D1-A): track 0.00 -> 30.1 mm, vias 0 -> 2
- net MID2: track 0.00 -> 29.5 mm, vias 0 -> 1
- net SLED: track 0.00 -> 28.7 mm, vias 0 -> 2
- net Net-(D3-K): track 0.00 -> 19.8 mm
- net IDDown: track 0.00 -> 19.5 mm
- net Net-(D10-K): track 0.00 -> 18.5 mm
- net Net-(D10-A): track 0.00 -> 15.4 mm
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- added copper zone on B.Cu, net GND
- added copper zone on F.Cu, net GND

Commit message: koi
Parts:
- U1: footprint XIAO:XIAO-ESP32C3-DIP -> XIAO:XIAO-ESP32C3-SMD; moved to B.Cu
- moved D12 46.7 mm to (55.3, 60.6), turned to -107 degrees
- moved D11 42.1 mm to (57.4, 61.2), turned to -105 degrees
- moved D10 37.5 mm to (59.5, 61.8), turned to -104 degrees
- moved SW2 35.8 mm to (99.8, 51.1), turned to 27 degrees
- moved R6 35.2 mm to (62.4, 58.7), turned to 77.5 degrees
- moved D9 32.9 mm to (61.6, 62.2), turned to -102.5 degrees
- moved R5 31.2 mm to (64.5, 59.1), turned to 80 degrees
- moved SW1 30.8 mm to (96.3, 44.6), turned to 27 degrees
- moved SW3 28.5 mm to (70.5, 46.8)
- moved D8 28.3 mm to (63.8, 62.7), turned to -100 degrees
- moved R4 27.3 mm to (66.5, 59.4), turned to 82 degrees
- moved D14 24.8 mm to (51.5, 42.3), turned to -90 degrees
- moved D7 23.7 mm to (65.9, 63.0), turned to -98 degrees
- moved U1 22.8 mm to (96.7, 45.0), turned to 27 degrees
- moved D1 21.1 mm to (77.4, 63.2), turned to 100 degrees
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Routing:
- net SID3: track 36.3 -> 0.00 mm, vias 1 -> 0
- net SID2: track 35.0 -> 0.00 mm, vias 1 -> 0
- net Net-(D1-K): track 34.5 -> 0.00 mm, vias 2 -> 0
- net SID1: track 33.6 -> 0.00 mm, vias 1 -> 0
- net MID3: track 33.4 -> 0.00 mm, vias 1 -> 0
- net MID1: track 32.5 -> 0.00 mm, vias 1 -> 0
- net Net-(D11-K): track 31.6 -> 0.00 mm
- net Action: track 30.8 -> 0.00 mm
- net Net-(D1-A): track 30.1 -> 0.00 mm, vias 2 -> 0
- net MID2: track 29.5 -> 0.00 mm, vias 1 -> 0
- net SLED: track 28.7 -> 0.00 mm, vias 2 -> 0
- net Net-(D3-K): track 19.8 -> 0.00 mm
- net IDDown: track 19.5 -> 0.00 mm
- net Net-(D10-K): track 18.5 -> 0.00 mm
- net Net-(D10-A): track 15.4 -> 0.00 mm
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Other:
- board size 54 x 38.5 mm -> 81.7 x 39.6 mm
- board text added: "ACTION"
- board text added: "CALL ID"
- board text added: "MY ID"
- board text added: "RCV"
- board text added: "SND"

Commit message: componentsPlacing
Parts:
- moved D13 29.5 mm to (80.7, 55.4), turned to -155 degrees
- moved R10 27.4 mm to (83.2, 48.7), turned to 100 degrees
- moved R7 27.4 mm to (83.2, 52.3), turned to 80 degrees
- moved SW3 24.4 mm to (93.7, 39.1), turned to 27 degrees
- moved D14 19.1 mm to (65.1, 55.8), turned to -10 degrees
- moved R8 14.0 mm to (61.5, 54.1), turned to 150 degrees
- moved R9 11.9 mm to (62.2, 52.9), turned to -30 degrees
- moved R4 7.62 mm to (73.8, 57.4), turned to 120 degrees
- moved R3 7.52 mm to (76.8, 52.1), turned to -175 degrees
- moved R6 7.32 mm to (69.7, 57.8), turned to 75 degrees
- moved R5 7.19 mm to (71.6, 58.0), turned to 90 degrees
- moved R2 5.39 mm to (76.4, 54.3), turned to 158 degrees
- moved R1 3.86 mm to (75.4, 56.0), turned to 142 degrees
Other:
- outline, holes or cut-outs redrawn
- board text added: "A"
- board text added: "ACT"
- board text added: "E"
- board text added: "G"
- board text added: "I"
- board text added: "L"
- board text added: "M"
- board text added: "O"
- board text added: "P"
- board text added: "R"
- board text removed: "ACTION"

Commit message: finishPCB
Parts:
- D1, D10, D11, D12, D13, D14, D2, D3, D4, D5, D6, D7, D8, D9: footprint LED_SMD:LED_0805_2012Metric_Pad1.15x1.40mm_HandSolder -> Extra:LED_0805_2012Metric_Pad1.15x1.40mm_HandSolder
- moved R1 21.9 mm to (63.8, 74.6)
- moved R10 21.9 mm to (71.6, 67.3)
- moved R2 21.9 mm to (64.8, 72.9)
- moved R7 21.9 mm to (71.6, 70.9)
- moved SW3 21.9 mm to (82.1, 57.7)
- moved U1 21.9 mm to (85.1, 63.6)
- moved D14 21.9 mm to (53.5, 74.3)
- moved R5 21.9 mm to (60.0, 76.6)
- moved R6 21.9 mm to (58.1, 76.4)
- moved D13 21.9 mm to (69.1, 73.9)
- moved R3 21.9 mm to (65.2, 70.7)
- moved R4 21.9 mm to (62.2, 76.0)
- moved R8 21.9 mm to (49.9, 72.7)
- moved R9 21.9 mm to (50.7, 71.4)
- moved SW1 21.9 mm to (84.8, 63.2)
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Connections:
- U1 pad 1: MID1 -> MID3
- U1 pad 2: MID2 -> MID1
- U1 pad 3: MID3 -> MID2
Routing:
- net SLED: track 0.00 -> 45.9 mm, vias 0 -> 1
- net RLED: track 0.00 -> 37.0 mm, vias 0 -> 1
- net Net-(D10-A): track 0.00 -> 27.8 mm, vias 0 -> 3
- net Net-(D1-K): track 0.00 -> 26.6 mm, vias 0 -> 5
- net SID3: track 0.00 -> 26.0 mm, vias 0 -> 1
- net Net-(D11-K): track 0.00 -> 25.8 mm, vias 0 -> 4
- net SID2: track 0.00 -> 24.6 mm, vias 0 -> 1
- net SID1: track 0.00 -> 23.1 mm, vias 0 -> 1
- net Net-(D3-K): track 0.00 -> 23.1 mm, vias 0 -> 2
- net MID2: track 0.00 -> 22.7 mm, vias 0 -> 1
- net Net-(D1-A): track 0.00 -> 22.2 mm, vias 0 -> 5
- net Net-(D10-K): track 0.00 -> 21.5 mm, vias 0 -> 2
- net MID1: track 0.00 -> 20.8 mm, vias 0 -> 1
- net Action: track 0.00 -> 20.6 mm, vias 0 -> 1
- net MID3: track 0.00 -> 19.4 mm, vias 0 -> 1
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Other:
- outline, holes or cut-outs redrawn

Commit message: qrcode and morsecode
Other:
- board text added: "A .- B -... C -.-. D -.. E . F ..-. G --. H .... I .. J .--- K -.- L .-.. M -- N -. O --- P .--. Q --.- R .-. S ... T - U ..- V ...- W .-- X -..- Y -.-- Z --.. 0 ----- 1 .---- 2 ..--- 3 ...-- 4 ....- 5 ..... 6 -.... 7 --... 8 ---.. 9 ----."

Commit message: finishPCB
Routing:
- net SID1: track 23.1 -> 22.6 mm
