File: pegoku-badge-pcb/pegoku-badge-pcb.kicad_pcb (KiCad board)
At the start: 2 copper layers, 81.7 x 39.6 mm, 28 parts, among them SW1 TS-1187A-B-A-B, SW2 TS-1187A-B-A-B, SW3 TS-1187A-B-A-B, U1 XIAO-ESP32-C3-DIP

Commit message: pegoku-badge
Other:
- board text added: "@Pegoku"
Changed lines of the file:
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@@
 		(property ki_fp_filters "LED* LED_SMD:* LED_THT:*")
 		(sheetname "/")
-		(sheetfile "badgePCB.kicad_sch")
+		(sheetfile "pegoku-badge-pcb.kicad_sch")
 		(units
 			(unit
@@
 		(property ki_fp_filters "LED* LED_SMD:* LED_THT:*")
 		(sheetname "/")
-		(sheetfile "badgePCB.kicad_sch")
+		(sheetfile "pegoku-badge-pcb.kicad_sch")
 		(units
 			(unit
@@
 		(property ki_fp_filters "R_*")
 		(sheetname "/")
-		(sheetfile "badgePCB.kicad_sch")
+		(sheetfile "pegoku-badge-pcb.kicad_sch")
 		(units
 			(unit
@@
 		(property ki_fp_filters "LED* LED_SMD:* LED_THT:*")
 		(sheetname "/")
-		(sheetfile "badgePCB.kicad_sch")
+		(sheetfile "pegoku-badge-pcb.kicad_sch")
 		(units
 			(unit
@@
 		(property ki_fp_filters "LED* LED_SMD:* LED_THT:*")
 		(sheetname "/")
-		(sheetfile "badgePCB.kicad_sch")
+		(sheetfile "pegoku-badge-pcb.kicad_sch")
 		(units
 			(unit
@@
 		(property ki_fp_filters "LED* LED_SMD:* LED_THT:*")
 		(sheetname "/")
-		(sheetfile "badgePCB.kicad_sch")
+		(sheetfile "pegoku-badge-pcb.kicad_sch")
 		(units
 			(unit
@@
 		(property ki_fp_filters "R_*")
 		(sheetname "/")
-		(sheetfile "badgePCB.kicad_sch")
+		(sheetfile "pegoku-badge-pcb.kicad_sch")
 		(units
 			(unit
@@
 		(property ki_fp_filters "R_*")
 		(sheetname "/")
-		(sheetfile "badgePCB.kicad_sch")
+		(sheetfile "pegoku-badge-pcb.kicad_sch")
 		(units
 			(unit
@@
 		(property ki_fp_filters "LED* LED_SMD:* LED_THT:*")
 		(sheetname "/")
-		(sheetfile "badgePCB.kicad_sch")
+		(sheetfile "pegoku-badge-pcb.kicad_sch")
 		(units
 			(unit
@@
 		(property ki_fp_filters "LED* LED_SMD:* LED_THT:*")
 		(sheetname "/")
-		(sheetfile "badgePCB.kicad_sch")
+		(sheetfile "pegoku-badge-pcb.kicad_sch")
 		(units
 			(unit
@@
 		(property ki_fp_filters "R_*")
 		(sheetname "/")
-		(sheetfile "badgePCB.kicad_sch")
+		(sheetfile "pegoku-badge-pcb.kicad_sch")
 		(units
 			(unit
@@
 		(property ki_fp_filters "R_*")
 		(sheetname "/")
-		(sheetfile "badgePCB.kicad_sch")
+		(sheetfile "pegoku-badge-pcb.kicad_sch")
 		(units
 			(unit
@@
 		(property ki_fp_filters "LED* LED_SMD:* LED_THT:*")
 		(sheetname "/")
-		(sheetfile "badgePCB.kicad_sch")
+		(sheetfile "pegoku-badge-pcb.kicad_sch")
 		(units
 			(unit
@@
 		(property ki_fp_filters "LED* LED_SMD:* LED_THT:*")
 		(sheetname "/")
-		(sheetfile "badgePCB.kicad_sch")
+		(sheetfile "pegoku-badge-pcb.kicad_sch")
 		(units
 			(unit
@@
 		)
 		(sheetname "/")
-		(sheetfile "badgePCB.kicad_sch")
+		(sheetfile "pegoku-badge-pcb.kicad_sch")
 		(units
 			(unit
@@
 		(property ki_fp_filters "LED* LED_SMD:* LED_THT:*")
 		(sheetname "/")
-		(sheetfile "badgePCB.kicad_sch")
+		(sheetfile "pegoku-badge-pcb.kicad_sch")
 		(units
 			(unit
@@
 		(property ki_fp_filters "R_*")
 		(sheetname "/")
-		(sheetfile "badgePCB.kicad_sch")
+		(sheetfile "pegoku-badge-pcb.kicad_sch")
 		(units
 			(unit
@@
 		(property ki_fp_filters "LED* LED_SMD:* LED_THT:*")
 		(sheetname "/")
-		(sheetfile "badgePCB.kicad_sch")
+		(sheetfile "pegoku-badge-pcb.kicad_sch")
 		(units
 			(unit
@@
 		(property ki_fp_filters "LED* LED_SMD:* LED_THT:*")
 		(sheetname "/")
-		(sheetfile "badgePCB.kicad_sch")
+		(sheetfile "pegoku-badge-pcb.kicad_sch")
 		(units
 			(unit
@@
 		(property ki_fp_filters "R_*")
 		(sheetname "/")
-		(sheetfile "badgePCB.kicad_sch")
+		(sheetfile "pegoku-badge-pcb.kicad_sch")
 		(units
 			(unit
@@
 		(property ki_fp_filters "R_*")
 		(sheetname "/")
-		(sheetfile "badgePCB.kicad_sch")
+		(sheetfile "pegoku-badge-pcb.kicad_sch")
 		(units
 			(unit
@@
 		(property ki_fp_filters "LED* LED_SMD:* LED_THT:*")
 		(sheetname "/")
-		(sheetfile "badgePCB.kicad_sch")
+		(sheetfile "pegoku-badge-pcb.kicad_sch")
 		(units
 			(unit
@@
 		(property ki_fp_filters "LED* LED_SMD:* LED_THT:*")
 		(sheetname "/")
-		(sheetfile "badgePCB.kicad_sch")
+		(sheetfile "pegoku-badge-pcb.kicad_sch")
 		(units
 			(unit
@@
 		)
 		(sheetname "/")
-		(sheetfile "badgePCB.kicad_sch")
+		(sheetfile "pegoku-badge-pcb.kicad_sch")
 		(units
 			(unit
@@
 		(property ki_fp_filters "R_*")
 		(sheetname "/")
-		(sheetfile "badgePCB.kicad_sch")
+		(sheetfile "pegoku-badge-pcb.kicad_sch")
 		(units
 			(unit
@@
 		(property ki_fp_filters "R_*")
 		(sheetname "/")
-		(sheetfile "badgePCB.kicad_sch")
+		(sheetfile "pegoku-badge-pcb.kicad_sch")
 		(units
 			(unit
@@
 		)
 		(sheetname "/")
-		(sheetfile "badgePCB.kicad_sch")
+		(sheetfile "pegoku-badge-pcb.kicad_sch")
 		(units
 			(unit
@@
 		)
 		(sheetname "/")
-		(sheetfile "badgePCB.kicad_sch")
+		(sheetfile "pegoku-badge-pcb.kicad_sch")
 		(units
 			(unit
@@
 		(layer "Edge.Cuts")
 	)
+	(gr_text "@Pegoku"
+		(at 63.85 52.775 -6)
+		(layer "F.SilkS")
+		(effects
+			(font
+				(size 1 1)
+				(thickness 0.15)
+				(bold yes)
+			)
+			(justify left bottom)
+		)
+	)
 	(gr_text "P"
-		(at 62.102796 54.528659 0)
+		(at 62.3 54.675 -3.4)
 		(layer "F.SilkS")
 		(effects
@@
 	)
 	(gr_text "E"
-		(at 63.152796 54.928659 0)
+		(at 63.2 54.975 -3)
 		(layer "F.SilkS")
 		(effects
@@
 	)
 	(gr_text "R"
-		(at 64.102796 55.128659 0)
+		(at 64.102796 55.128659 -2.5)
 		(layer "F.SilkS")
 		(effects
@@
 	)
 	(gr_text "E"
-		(at 65.152796 55.328659 0)
+		(at 65.15 55.35 -2)
 		(layer "F.SilkS")
 		(effects
