File: raghav-fallout-badge/raghav-fallout-badge.kicad_pcb (KiCad board)
At the start: 2 copper layers, 68.1 x 82.8 mm, 29 parts, among them SW1 TS-1187A-B-A-B, SW2 TS-1187A-B-A-B, SW3 TS-1187A-B-A-B, U1 XIAO-ESP32-C3-DIP

Commit message: fix
Other:
- board text added: "Designed by: @Pegoku"
Changed lines of the file:
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@@
 		(duplicate_pad_numbers_are_jumpers no)
 		(fp_line
-			(start -0.254725 0.522501)
+			(start -0.254725 0.522502)
 			(end 0.254725 0.522501)
 			(stroke
@@
 		(fp_line
 			(start -0.254725 -0.522501)
-			(end 0.254725 -0.522501)
+			(end 0.254725 -0.522502)
 			(stroke
 				(width 0.12)
@@
 		(fp_poly
 			(pts
-				(xy 0.8 -0.4125) (xy 0.8 0.412499) (xy -0.8 0.4125) (xy -0.8 -0.412499)
+				(xy 0.800001 -0.4125) (xy 0.8 0.412499) (xy -0.800001 0.4125) (xy -0.8 -0.412499)
 			)
 			(stroke
@@
 		)
 	)
+	(gr_text "Designed by: @Pegoku"
+		(at 113.55 174.425 -0)
+		(layer "B.SilkS")
+		(effects
+			(font
+				(size 1 1)
+				(thickness 0.15)
+			)
+			(justify left bottom mirror)
+		)
+	)
